File: Hardware/London_EPS-v.2.0/London_EPS-v.2.0.brd (EAGLE design)
At the start: 86 x 86 mm, 60 parts, among them IC1 LM2596S-5.0_NOPB, IC2 LM2596SX-3.3_NOPB, IC3 LT3652HVEMSE#PBF, IC4 LM234DT, IC5 TLV810EA29DBZR, IC6 INA3221AIRGVT

Commit message: Add files via upload
Parts:
- moved D6 0.95 mm to (29.8, 50.8)
- moved R10 0.95 mm to (36.2, 50.8)
- moved C7 0.63 mm to (36.2, 47.3)
- moved D4 0.63 mm to (29.8, 47.3)
- moved C6 0.32 mm to (29.8, 44.5)
- moved R13 0.32 mm to (36.2, 44.5)
- renumbered STACK to PILHA
Routing:
- net GND: track 31.2 -> 87.9 mm, vias 24 -> 41
- net 5V+: track 83.2 -> 93.2 mm
- net 3V3+: track 96.4 -> 104.8 mm, vias 2 -> 4
- net N$30: track 6.59 -> 5.00 mm
- net BAT+: track 223.7 -> 222.1 mm
- net N$23: track 31.6 -> 32.2 mm
- net 3V3: track 220.1 -> 219.5 mm
