File: Hardware/London_EPS-v.2.0/London_EPS-v.2.0.sch (EAGLE design)
At the start: 60 parts, among them IC1 LM2596S-5.0_NOPB, IC2 LM2596SX-3.3_NOPB, IC3 LT3652HVEMSE#PBF, IC4 LM234DT, IC5 TLV810EA29DBZR, IC6 INA3221AIRGVT

Commit message: Add files via upload
Parts:
- renumbered STACK to PILHA
Other:
- note added: "Pilha"
- note removed: "Conector da Stack"
