File: Hardware/Ribatski_EPS-v.2.0/Ribatski_EPS-v2.0.sch (EAGLE design)
At the start: 37 parts, among them IC1 MAX17205G+T, Q1 4N25-300E, Q2 BSC010NE2LS

Commit message: Add files via upload
Parts:
- removed Q2: BSC010NE2LS, SamacSys_Parts:BSC010NE2LS
- removed R10: 0, rcl:R-EU_R0805
- removed R7: 1k, rcl:R-EU_R0805
- removed R8: 10k, rcl:R-EU_R0805
- Q1: value 4N25-300E -> BSC010NE2LS; device SamacSys_Parts:4N25-300E -> SamacSys_Parts:BSC010NE2LS
- R5: value 0 -> 1.3
- R6: value 100 -> 10k
- renumbered STACK to PILHA
Connections:
- removed net N$10: Q2.S_1, Q2.S_2, Q2.S_3, U$2.P$2
- removed net N$11: Q2.D_1, Q2.D_2, Q2.D_3, Q2.D_4, R5.1
- removed net N$12: Q2.G, R10.2
- removed net N$8: Q1.ANODE, R6.2, R7.1
- removed net N$9: Q1.COLLECTOR, R10.1, R8.1
- new net N$5: Q1.G, R5.2, R6.2
- new net RL: Q1.D_1, Q1.D_2, Q1.D_3, Q1.D_4, U$2.P$1
- net 3S: now also U$2.P$2; no longer R5.2, R8.2
- net 3V3: no longer R7.2
- net GND: now also Q1.S_1, Q1.S_2, Q1.S_3, R6.1; no longer Q1.CATHODE, Q1.EMITTER, U$2.P$1
- net PWM: now also R5.1; no longer R6.1
Other:
- note added: "Conexões"
- note removed: "Conector da stack"
- moved on the sheet: R5, R6
