File: Hardware/Ribatski_EPS-v.2.0/Ribatski_EPS-v2.0.brd (EAGLE design)
At the start: 86 x 86 mm, 37 parts, among them IC1 MAX17205G+T, Q1 4N25-300E, Q2 BSC010NE2LS

Commit message: Add files via upload
Parts:
- removed Q2: BSC010NE2LS, SamacSys_Parts:PG-TDSON-8
- removed R10: 0, rcl:R0805
- removed R7: 1k, rcl:R0805
- removed R8: 10k, rcl:R0805
- Q1: value 4N25-300E -> BSC010NE2LS; device SamacSys_Parts:SOP254P1016X400-6N -> SamacSys_Parts:PG-TDSON-8
- R5: value 0 -> 1.3
- R6: value 100 -> 10k
- moved R6 28.6 mm to (58.4, 56.7), turned to 0 degrees
- moved Q1 27.0 mm to (58.4, 65.2), turned to 0 degrees
- moved R5 3.35 mm to (58.4, 54.1), turned to 0 degrees
- moved D4 2.86 mm to (58.4, 50.8), flipped to the top, turned to 180 degrees
- renumbered STACK to PILHA
Connections:
- removed net N$10: Q2.1, Q2.2, Q2.3, U$2.P$2
- removed net N$11: Q2.5, Q2.6, Q2.7, Q2.8, R5.1
- removed net N$12: Q2.4, R10.2
- removed net N$8: Q1.1, R6.2, R7.1
- removed net N$9: Q1.5, R10.1, R8.1
- new net N$5: Q1.4, R5.2, R6.2
- new net RL: Q1.5, Q1.6, Q1.7, Q1.8, U$2.P$1
- net 3S: now also U$2.P$2; no longer R5.2, R8.2
- net 3V3: no longer R7.2
- net GND: now also Q1.1, Q1.3, R6.1; no longer Q1.4, U$2.P$1
- net PWM: now also R5.1; no longer R6.1
Routing:
- net N$10: track 31.5 -> 0.00 mm
- net 3S: track 184.8 -> 156.5 mm, vias 0 -> 2
- net RL: track 0.00 -> 25.6 mm
- net PWM: track 129.0 -> 107.3 mm, vias 4 -> 7
- net GND: track 21.2 -> 35.4 mm, vias 14 -> 49
- net N$11: track 11.2 -> 0.00 mm
- net N$9: track 5.74 -> 0.00 mm
- net N$8: track 5.74 -> 0.00 mm
- net N$5: track 0.00 -> 5.51 mm
- net N$20: track 15.4 -> 12.4 mm
- net 3V3: track 110.1 -> 107.2 mm
- net N$12: track 2.79 -> 0.00 mm
- net N$18: track 69.2 -> 71.8 mm, vias 1 -> 2
- net BAT+: track 88.6 -> 86.5 mm, vias 1 -> 3
- net SCL2: track 117.8 -> 116.5 mm
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
Commit message: Add files via upload
Parts:
- moved R2 0.72 mm to (25.1, 68.6)
- moved BT1 0.64 mm to (43.0, 58.6)
- moved R12 0.48 mm to (43.0, 48.5)
- moved R3 0.48 mm to (24.8, 48.4)
- moved BT2 0.32 mm to (43.0, 38.3)
- moved R11 0.16 mm to (43.0, 28.2)
- moved R13 0.16 mm to (32.7, 28.1)
- moved R4 0.16 mm to (24.8, 28.1)
- moved R9 0.16 mm to (12.4, 28.2)
Routing:
- net 3V3: track 107.2 -> 104.2 mm
- net GND: track 35.4 -> 38.3 mm
- net 3S: track 156.5 -> 154.5 mm
- net 2S: track 171.2 -> 172.5 mm
- net ALRT1: track 140.9 -> 142.0 mm
- net SDA2: track 105.1 -> 104.5 mm
- net N$16: track 79.2 -> 79.7 mm
